Commit message: Então toma.

File: denso_robot_ros2/denso_robot_description/urdf/denso_robot/denso_robot_macro.ros2_control.xacro (robot description, xacro)
@@ -1,8 +1,9 @@
 <?xml version="1.0" encoding="UTF-8"?>
 <robot xmlns:xacro="http://www.ros.org/wiki/xacro">
-  <xacro:macro name="denso_robot_ros2_control" params="name prefix
+ <xacro:macro name="denso_robot_ros2_control" params="name prefix
     use_fake_hardware:=^|false mock_sensor_commands:=^|false
     sim_gazebo_classic:=^|false
-    sim_gazebo:=^|true
+    sim_gazebo:=^|false
+    isaac:=^|true
     robot_ip:=^|192.168.0.1
     robot_port:=^|5007
@@ -25,5 +26,10 @@
           <param name="state_following_offset">0.0</param>
         </xacro:if>
-        <xacro:unless value="${use_fake_hardware or sim_gazebo_classic or sim_gazebo}">
+        <xacro:if value="${isaac}">
+          <plugin>topic_based_ros2_control/TopicBasedSystem</plugin>
+          <param name="joint_states_topic">/joint_states</param>
+          <param name="joint_commands_topic">/joint_commands</param>
+        </xacro:if>
+        <xacro:unless value="${use_fake_hardware or sim_gazebo_classic or sim_gazebo or isaac}">
           <plugin>denso_hw/denso_hw</plugin>
           <param name="robot_ip">${robot_ip}</param>

File: denso_robot_ros2/denso_robot_description/urdf/denso_robot/denso_robot_macro.xacro (robot description, xacro)
@@ -1,16 +1,21 @@
 <?xml version="1.0" encoding="UTF-8"?>
 <robot xmlns:xacro="http://wiki.ros.org/xacro">
+  <!-- Inclui definições comuns -->
   <xacro:include filename="$(find denso_robot_description)/urdf/common.xacro" />
+  <!-- Propriedade que controla o modo -->
+  <!-- mode=0 -> usa o mesh J6.dae -->
+  <!-- mode=1 -> usa o cilindro -->
   <xacro:macro name="denso_robot" params="
     prefix
     parent
     *origin
+    mode
     initial_positions:=${dict(joint1=0.0,joint2=0.0,joint3=1.57,joint4=0.0,joint5=0.0,joint6=0.0)}"
-    >
-    <!-- LINKS -->
+  >
+    <!-- =========================== -->
+    <!-- ======== LINKS ============ -->
+    <!-- =========================== -->
     <!-- base link -->
     <link name="${prefix}base_link">
-      <!-- Default inertial for Gazebo/Ingnition - copy and edit block from 'common.xacro'
-           to get more realistic behaviour-->
       <xacro:default_inertial/>
       <visual>
@@ -27,8 +32,6 @@
       </collision>
     </link>
-    <!-- link 1 -->
+    <!-- link1 -->
     <link name="${prefix}link1">
-      <!-- Default inertial for Gazebo/Ingnition - copy and edit block from 'common.xacro'
-           to get more realistic behaviour-->
       <xacro:default_inertial/>
       <visual>
@@ -45,8 +48,6 @@
       </collision>
     </link>
-    <!-- link 2 -->
+    <!-- link2 -->
     <link name="${prefix}link2">
-      <!-- Default inertial for Gazebo/Ingnition - copy and edit block from 'common.xacro'
-           to get more realistic behaviour-->
       <xacro:default_inertial/>
       <visual>
@@ -59,12 +60,10 @@
         <origin xyz="0 0 0" rpy="0 0 0" />
         <geometry>
-          <mesh filename="package://denso_robot_description/meshes/denso_robot/visual/J2.dae"  />
-        </geometry>
-      </collision>
-    </link>
-    <!-- link 3 -->
+          <mesh filename="package://denso_robot_description/meshes/denso_robot/visual/J2.dae" />
+        </geometry>
+      </collision>
+    </link>
+    <!-- link3 -->
     <link name="${prefix}link3">
-      <!-- Default inertial for Gazebo/Ingnition - copy and edit block from 'common.xacro'
-           to get more realistic behaviour-->
       <xacro:default_inertial/>
       <visual>
@@ -77,12 +76,10 @@
         <origin xyz="0 0 0" rpy="0 0 0" />
         <geometry>
-          <mesh filename="package://denso_robot_description/meshes/denso_robot/visual/J3.dae"  />
-        </geometry>
-      </collision>
-    </link>
-    <!-- link 4 -->
+          <mesh filename="package://denso_robot_description/meshes/denso_robot/visual/J3.dae" />
+        </geometry>
+      </collision>
+    </link>
+    <!-- link4 -->
     <link name="${prefix}link4">
-      <!-- Default inertial for Gazebo/Ingnition - copy and edit block from 'common.xacro'
-           to get more realistic behaviour-->
       <xacro:default_inertial/>
       <visual>
@@ -95,12 +92,10 @@
         <origin xyz="0 0 0" rpy="0 0 0" />
         <geometry>
-          <mesh filename="package://denso_robot_description/meshes/denso_robot/visual/J4.dae"  />
-        </geometry>
-      </collision>
-    </link>
-    <!-- link 5 -->
+          <mesh filename="package://denso_robot_description/meshes/denso_robot/visual/J4.dae" />
+        </geometry>
+      </collision>
+    </link>
+    <!-- link5 -->
     <link name="${prefix}link5">
-      <!-- Default inertial for Gazebo/Ingnition - copy and edit block from 'common.xacro'
-           to get more realistic behaviour-->
       <xacro:default_inertial/>
       <visual>
@@ -117,28 +112,51 @@
       </collision>
     </link>
-    <!-- link 6 -->
-    <link name="${prefix}link6">
-      <!-- Default inertial for Gazebo/Ingnition - copy and edit block from 'common.xacro'
-           to get more realistic behaviour-->
-      <xacro:default_inertial/>
-      <visual>
-        <origin xyz="0 0 0" rpy="0 0 0" />
-        <geometry>
-          <mesh filename="package://denso_robot_description/meshes/denso_robot/visual/J6.dae" />
-        </geometry>
-      </visual>
-      <collision>
-        <origin xyz="0 0 0" rpy="0 0 0" />
-        <geometry>
-          <mesh filename="package://denso_robot_description/meshes/denso_robot/visual/J6.dae" />
-        </geometry>
-      </collision>
-    </link>
-    <!-- All-zero tool frame. This frame should correspond to the TOOL frame of the robot's controller.) -->
+    <!-- ========================== -->
+    <!-- link6 - alterna por 'mode' -->
+    <!-- ========================== -->
+    <xacro:if value="${mode == 0}">
+      <link name="${prefix}link6">
+        <xacro:default_inertial/>
+        <visual>
+          <origin xyz="0 0 0" rpy="0 0 0" />
+          <geometry>
+            <mesh filename="package://denso_robot_description/meshes/denso_robot/visual/J6.dae" />
+          </geometry>
+        </visual>
+        <collision>
+          <origin xyz="0 0 0" rpy="0 0 0" />
+          <geometry>
+            <mesh filename="package://denso_robot_description/meshes/denso_robot/visual/J6.dae" />
+          </geometry>
+        </collision>
+      </link>
+    </xacro:if>
+    <xacro:if value="${mode == 1}">
+      <link name="${prefix}link6">
+        <xacro:default_inertial/>
+        <inertial>
+          <origin xyz="0.0 0.0 0.0" rpy="0.0 0.0 0.0"/>
+          <mass value="1.0"/>
+          <inertia ixx="0.00015" ixy="0.0" ixz="0.0" iyy="0.0009083" iyz="0.0" izz="0.0009083"/>
+        </inertial>
+        <visual>
+          <origin xyz="0.0 0.0 0.09" rpy="0.0 0.0 0.0"/>
+          <geometry>
+            <cylinder radius="0.015" length="0.2"/>
+          </geometry>
+        </visual>
+        <collision>
+          <origin xyz="0.0 0.0 0.09" rpy="0.0 0.0 0.0"/>
+          <geometry>
+            <cylinder radius="0.015" length="0.2"/>
+          </geometry>
+        </collision>
+      </link>
+    </xacro:if>
+    <!-- tool0 -->
     <link name="${prefix}tool0" />
-    <!-- tool link -->
-    <!-- END LINKS -->
-    <!-- JOINTS -->
-    <!-- base_joint fixes base_link to the environment -->
+    <!-- =========================== -->
+    <!-- ======== JOINTS =========== -->
+    <!-- =========================== -->
     <joint name="${prefix}base_joint" type="fixed">
       <xacro:insert_block name="origin" />
@@ -146,5 +164,4 @@
       <child link="${prefix}base_link" />
     </joint>
-    <!-- joint 1 -->
     <joint name="${prefix}joint1" type="revolute">
       <origin xyz="0 0 0.197500" rpy="0 0 0" />
@@ -155,5 +172,4 @@
       <dynamics damping="0.7" friction="0.0"/>
     </joint>
-    <!-- joint 2 -->
     <joint name="${prefix}joint2" type="revolute">
       <origin xyz="0.03 0 0.1975" rpy="0 0 0" />
@@ -164,5 +180,4 @@
       <dynamics damping="0.7" friction="0.0"/>
     </joint>
-    <!-- joint 3 -->
     <joint name="${prefix}joint3" type="revolute">
       <origin xyz="0 0 0.445" rpy="0 0 0" />
@@ -173,5 +188,4 @@
       <dynamics damping="0.7" friction="0.0"/>
     </joint>
-    <!-- joint 4 -->
     <joint name="${prefix}joint4" type="revolute">
       <origin xyz="-0.02 0 0.287" rpy="0 0 0" />
@@ -182,5 +196,4 @@
       <dynamics damping="0.7" friction="0.0"/>
     </joint>
-    <!-- joint 5 -->
     <joint name="${prefix}joint5" type="revolute">
       <origin xyz="0 0 0.143" rpy="0 0 0" />
@@ -191,14 +204,24 @@
       <dynamics damping="0.7" friction="0.0"/>
     </joint>
-    <!-- joint 6 -->
-    <joint name="${prefix}joint6" type="revolute">
-      <origin xyz="0 0 0.08" rpy="0 0 0" />
-      <parent link="${prefix}link5" />
-      <child link="${prefix}link6" />
-      <axis xyz="0 0 1" />
-      <limit effort="1000" lower="${radians(-360)}" upper="${radians(360)}" velocity="${radians(864)}" />
-      <dynamics damping="0.7" friction="0.0"/>
-    </joint>
-    <!-- tool frame - fixed frame -->
+    <xacro:if value="${mode == 0}">
+      <joint name="${prefix}joint6" type="revolute">
+        <origin xyz="0 0 0.08" rpy="0 0 0" />
+        <parent link="${prefix}link5" />
+        <child link="${prefix}link6" />
+        <axis xyz="0 0 1" />
+        <limit effort="1000" lower="${radians(-360)}" upper="${radians(360)}" velocity="${radians(864)}" />
+        <dynamics damping="0.7" friction="0.0"/>
+      </joint>
+    </xacro:if>
+    <xacro:if value="${mode == 1}">
+      <joint name="${prefix}joint6" type="revolute">
+        <origin xyz="0 0 0.26" rpy="0 ${pi} 0" />
+        <parent link="${prefix}link5" />
+        <child link="${prefix}link6" />
+        <axis xyz="0 0 1" />
+        <limit effort="1000" lower="${radians(-360)}" upper="${radians(360)}" velocity="${radians(864)}" />
+        <dynamics damping="0.7" friction="0.0"/>
+      </joint>
+    </xacro:if>
     <joint name="${prefix}joint6-tool0" type="fixed">
       <parent link="${prefix}link6" />
@@ -206,5 +229,4 @@
       <origin xyz="0 0 -0.115" rpy="0 ${-pi} ${-pi/2}" />
     </joint>
-    <!-- END JOINTS -->
   </xacro:macro>
 </robot>
